File: chaotist/pcb/chaotist.kicad_pcb (KiCad board)
At the start: 2 copper layers, 229.3 x 91.2 mm, 105 parts, among them SW1 Reset, U1 Raspberry_Pi_Pico

Commit message: updated pcb; added initial code
Parts:
- moved REF** 1.35 mm to (143.1, 106.4)
- moved D37a1 0.93 mm to (140.4, 102.2)
Routing:
- net R1: track 201.9 -> 197.7 mm
- net R0: track 227.4 -> 224.7 mm
- net C3: track 156.0 -> 154.5 mm
- net Net-(D17-A): track 14.6 -> 15.2 mm
- net C6: track 55.1 -> 55.7 mm
- net Net-(D37a1-A): track 7.18 -> 6.67 mm
Other:
- board text added: "1x 2.75u (S1) + stab or 1.5u+1.25u (S1a1+S1b1)"
- board text added: "1x 2.75u (S12) + stab or 1.5u+1.25u (S12a1+S12b1)"
- board text removed: "1x 2.75u (S1) + stab or 1.25u+1.5u (S1a1+S1b1)"
- board text removed: "1x 2.75u (S12) + stab or 1.25u+1.5u (S12a1+S12b1)"

Commit message: final version for production
Connections:
- U1 pad 33: unconnected-(U1-AGND-Pad33) -> GND
Routing:
- net GND: track 26.1 -> 0.08 mm
