File: chaotist/pcb/chaotist.kicad_sch (KiCad schematic)
At the start: 90 parts, among them SW1 Reset, U1 Raspberry_Pi_Pico

Commit message: final version for production
Connections:
- net GND: now also U1.33 (AGND)
Changed lines of the file:
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@@
+    )
+  )
+  (global_label "GND" (shape input) (at 274.32 45.72 0) (fields_autoplaced)
+    (effects (font (size 1.27 1.27)) (justify left))
+    (property "Intersheetrefs" "${INTERSHEET_REFS}" (at 281.1757 45.72 0)
+      (effects (font (size 1.27 1.27)) (justify left) hide)
     )
   )
